File: EAGLE/HEL Lasersysteem/Laser Centraal/Laser Centraal.sch (EAGLE design)
At the start: 82 parts, among them IC1 LMV324M, IC2 LMV324M, IC3 74LVC1G14DBV, IC6 ATMEGA328P-AU, IC7 FT232RL

Commit message: Laser PCB's aangepast
Parts:
- added BRES, OUTGND2: LSP10, solpad:LSP10
- added C17: 100n, rcl:C-EUC0805
- renumbered LED0UIT to LED0, LED1UIT to LED1, LED2UIT to LED2
Connections:
- net BUTTIN: now also IC6.PC4(ADC4/SDA); no longer IC6.PC5(ADC5/SCL)
- net BUTTOUT: now also IC6.PC5(ADC5/SCL); no longer IC6.PC4(ADC4/SDA)
- net GND: now also C17.2, OUTGND2.MP
- net N$15: now also BRES.MP
- net N$2: now also D4.A; no longer D2.A
- net N$4: now also D2.A; no longer D4.A
- net N$6: now also D8.A; no longer D6.A
- net N$8: now also D6.A; no longer D8.A
- net VCC: now also C17.1
Other:
- moved on the sheet: D2, D4, D6, D8

Commit message: tweede versie laser gerbers klaargemaakt voor bestelling
Parts:
- removed C14, C15, C9: 100nF, rcl:C-EUC0805
- removed D18: BAT60J, diode:BAT60J
- removed IC7: FT232RL, ftdichip:FT232RL
- removed MINI-USB-B: MINI_USB_B-KRHRO-SELECU-M-M5DS-W-4, mini USB B Korean Hroparts Elec U-M-M5DS-W-4:MINI_USB_B-KRHRO-SELECU-M-M5DS-W-4
- removed R27, R28: 1k, rcl:R-EU_R0805
- added R23: 100, rcl:R-EU_R0805
- added RX, TX: LSP10, solpad:LSP10
- C1: device rcl:C-EUC0805K -> rcl:C-EUC0805
- C8: value 4u7 -> 100n
Connections:
- removed net 3V3: C15.1, IC7.3V3OUT
- removed net N$19: IC7.USBDP, MINI-USB-B.D+
- removed net N$24: IC7.USBDM, MINI-USB-B.D-
- removed net RX: IC7.TXD, R28.2
- removed net TX: IC7.RXD, R27.2
- removed net VUSB: C8.1, C9.1, D18.A, MINI-USB-B.VBUS
- net D0/RX: now also RX.MP; no longer R28.1
- net D1/TX: now also TX.MP; no longer R27.1
- net GND: no longer C15.2, C9.2, IC7.GND, IC7.GND@1, IC7.GND@2, IC7.GND@A, IC7.TEST, MINI-USB-B.CASE, MINI-USB-B.GND
- net N$15: no longer BRES.MP
- net N$18: now also BRES.MP, R23.2; no longer C14.2, IC7.!DTR
- net RESET: now also R23.1; no longer C14.1
- net VCC: now also C8.1; no longer D18.C, IC7.VCC, IC7.VCCIO
Other:
- moved on the sheet: BRES, C8
