File: EAGLE/HEL Lasersysteem/Laser Zender/laser zender.brd (EAGLE design)
At the start: 20 x 32 mm, 18 parts, among them IC2 LM556D

Commit message: kleine aanpassingen
Parts:
- R6: value 100k -> 10k
Changed lines of the file:
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@@
 <drawing>
 <settings>
-<setting alwaysvectorfont="yes"/>
+<setting alwaysvectorfont="no"/>
 <setting verticaltext="up"/>
 </settings>
@@
 <attribute name="VALUE" x="9.652" y="1.778" size="1.27" layer="27" rot="R90"/>
 </element>
-<element name="R6" library="rcl" library_urn="urn:adsk.eagle:library:334" package="R0805" package3d_urn="urn:adsk.eagle:package:23553/2" value="100k" x="2.032" y="6.096" smashed="yes">
+<element name="R6" library="rcl" library_urn="urn:adsk.eagle:library:334" package="R0805" package3d_urn="urn:adsk.eagle:package:23553/2" value="10k" x="2.032" y="6.096" smashed="yes">
 <attribute name="NAME" x="1.524" y="7.112" size="0.8128" layer="25"/>
 <attribute name="SPICEPREFIX" value="R" x="2.032" y="6.096" size="1.778" layer="27" display="off"/>
